File: KiCad/Leviathan.kicad_sch (KiCad schematic)
At the start: 415 parts, among them J1 PWR_HV_DRV, J10 HV_Stepper1, J11 HV_Stepper0, J12 LED-Strip, J13 FAN_V, J14 FAN_V, J15 FAN_V, J16 FAN_V, J17 USB_C_Receptacle_USB2.0, J18 T2, J19 T3, J2 Stepper0, J20 PROBE_V, J21 Z-Probe, J22 FAN_0, J23 FAN_1, J24 FAN_2, J25 FAN_3, J26 T0, J27 T1, J28 Neopixel, J29 Fil, J3 Stepper1, J30 X, J31 Y, J32 Z, J33 CAN_BUS, J34 Conn_02x15_Odd_Even, J4 Stepper2, J5 Stepper3, J6 Stepper4, J7 PWR_IN, J8 SWD, J9 PWR/UART, Q1 SUD50P06-15-GE3, Q10 SiZ270DT, Q11 SiZ270DT, Q12 SiZ270DT, Q13 SQ2348ES, Q14 SQ2348ES, Q15 SQ2348ES, Q16 SQ2348ES, Q2 SUD50P06-15-GE3, Q3 SiZ270DT, Q4 SiZ270DT, Q5 DMTH6005LK3Q-13, Q6 SiZ270DT, Q7 SiZ270DT, Q8 DMTH6005LK3Q-13, Q9 SiZ270DT, SW1 Reset, SW2 BOOT0, U1 TMC2209_LA, U10 TMC5160-WA, U11 AP2112K-3.3V{slash}AP2127K-3.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, U12 TJA1051T-3, U13 RPi4, U14 USBLC6-2SC6, U15 74LVC1G17GW, U16 LM3407MY, U2 TMC2209_LA, U3 TMC2209_LA, U4 TMC2209_LA, U5 TMC2209_LA, U6 TMC5160-WA, U7 MCP1416, U8 MCP1416, U9 STM32F446ZET6, Y1 12MHz

Commit message: Updated KiCad files, schematic exported to pdf file
Other:
- note added: "https://github.com/MotorDynamicsLab/Leviathan"
Changed lines of the file:
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@@
   (title_block
     (title "Leviathan Mainboard")
-    (date "2021-10-03")
+    (date "2023-11-28")
     (rev "1.2")
     (company "Voron")
@@
     (effects (font (size 4 4) (thickness 0.8) bold italic) (justify left bottom))
   )
+  (text "https://github.com/MotorDynamicsLab/Leviathan" (at 504.825 396.24 0)
+    (effects (font (size 2 2)) (justify left bottom))
+  )
   (text "Ports" (at 96.52 349.25 0)
